Commit message: Ignore catkin_ws and commit workspace changes

File: ros2_ws/install/panda_description/share/panda_description/urdf/panda.urdf.xacro (robot description, xacro)
@@ -1 +1 @@
-/root/ros2_panda_ws/src/panda_description/urdf/panda.urdf.xacro
+/opt/ws_panda/src/panda_description/urdf/panda.urdf.xacro

File: ros2_ws/src/panda_description/urdf/panda.urdf.xacro (robot description, xacro)
@@ -1,51 +1,99 @@
-<?xml version="1.0" encoding="utf-8"?>
-<robot xmlns:xacro="http://www.ros.org/wiki/xacro" name="panda">
-  <!-- Pull Panda from MoveIt resources (apt: ros-humble-moveit-resources-panda-description) -->
-  <xacro:include filename="$(find moveit_resources_panda_description)/urdf/panda.urdf.xacro"/>
-  <!-- ======== Arguments you can expose to launches ======== -->
-  <xacro:arg name="arm_id" default="panda"/>
-  <!-- Classic Gazebo plugins don't work in Gazebo Harmonic; keep off -->
-  <xacro:arg name="use_gazebo_classic_plugins" default="false"/>
-  <xacro:arg name="use_gt_planning_scene" default="false"/>
-  <xacro:arg name="use_gt_bounding_box" default="false"/>
-  <xacro:arg name="enable_gt_joint_axis" default="false"/>
-  <!-- ======== Instantiate the Panda robot ======== -->
-  <!-- The MoveIt resource provides the Panda macros; the minimal, robust form is: -->
-  <xacro:franka_robot arm_id="$(arg arm_id)"/>
-  <!-- If you ever need to override joint limits explicitly, you can pass them like this:
-  <xacro:franka_robot
-      arm_id="$(arg arm_id)"
-      joint_limits="${xacro.load_yaml('$(find moveit_resources_panda_description)/config/joint_limits.yaml')}"/>
-  -->
-  <!-- ======== (Optional) Classic Gazebo plugins — disabled by default ======== -->
-  <!-- These were designed for Gazebo Classic. Keep them off for ros_gz_sim/Harmonic. -->
-  <xacro:if value="$(arg use_gazebo_classic_plugins)">
-    <gazebo>
-      <xacro:if value="$(arg use_gt_planning_scene)">
-        <plugin filename="libgazebo_ros_moveit_planning_scene.so" name="gazebo_ros_moveit_planning_scene">
-          <topicName>/planning_scene</topicName>
-          <updatePeriod>3.0</updatePeriod>
-        </plugin>
-      </xacro:if>
-      <xacro:if value="$(arg use_gt_bounding_box)">
-        <plugin filename="libgazebo_ros_bbox_3d_plugin.so" name="gazebo_ros_bbox_3d_plugin">
-          <links_to_publish>
-            <link>cabinet::drawer0</link>
-            <link>cabinet::drawer1</link>
-            <link>cabinet::drawer2</link>
-            <link>cabinet::drawer3</link>
-            <link>cabinet::handle_0</link>
-            <link>cabinet::handle_1</link>
-            <link>cabinet::handle_2</link>
-            <link>cabinet::handle_3</link>
-          </links_to_publish>
-        </plugin>
-      </xacro:if>
-      <xacro:if value="$(arg enable_gt_joint_axis)">
-        <plugin filename="libgazebo_ros_joint_axis_service.so" name="gazebo_ros_joint_axis_service">
-          <NodeName>gazebo_ros_joint_axis_service</NodeName>
-        </plugin>
-      </xacro:if>
-    </gazebo>
+<?xml version="1.0"?>
+<!-- URDF for Franka Emika Panda -->
+<robot xmlns:xacro="http://wiki.ros.org/xacro" name="$(arg name)">
+  <!--                   -->
+  <!-- Imported elements -->
+  <!--                   -->
+  <xacro:include filename="$(find panda_description)/urdf/panda_arm.xacro"/>
+  <xacro:include filename="$(find panda_description)/urdf/panda_gripper.xacro"/>
+  <xacro:include filename="$(find panda_description)/urdf/panda_utils.xacro"/>
+  <xacro:include filename="$(find panda_description)/urdf/panda.gazebo"/>
+  <!--            -->
+  <!-- Parameters -->
+  <!--            -->
+  <!-- Name of the robot (mandatory) -->
+  <xacro:arg name="name" default="panda"/>
+  <!-- Prefix for all entities -->
+  <xacro:arg name="prefix" default="$(arg name)_"/>
+  <!-- Flag to enable default gripper -->
+  <xacro:arg name="gripper" default="true" />
+  <!-- Flag to enable collision geometry for manipulator's arm -->
+  <xacro:arg name="collision_arm" default="true"/>
+  <!-- Flag to enable collision geometry for manipulator's gripper (hand and fingers) -->
+  <xacro:arg name="collision_gripper" default="true"/>
+  <!-- Flag to enable safety limits controllers on manipulator joints -->
+  <xacro:arg name="safety_limits" default="false"/>
+  <!-- Lower and upper margin for position limits of all safety controllers -->
+  <xacro:arg name="safety_position_margin" default="0.17453293"/>
+  <!-- Parametric k-position factor of all safety controllers -->
+  <xacro:arg name="safety_k_position" default="100.0"/>
+  <!-- Parametric k-velocity factor of all safety controllers -->
+  <xacro:arg name="safety_k_velocity" default="40.0"/>
+  <!-- Flag to enable ros2 controllers for manipulator -->
+  <xacro:arg name="ros2_control" default="true"/>
+  <!-- The ros2_control plugin that should be loaded for the manipulator ('fake', 'ign', 'real' or custom) -->
+  <xacro:arg name="ros2_control_plugin" default="ign"/>
+  <!-- The output control command interface provided by ros2_control ('position', 'velocity', 'effort' or certain combinations 'position,velocity') -->
+  <xacro:arg name="ros2_control_command_interface" default="effort"/>
+  <!-- The filepath to parameters of ROS 2 controllers -->
+  <xacro:arg name="ros2_controller_parameters" default="$(find panda_moveit_config)/config/controllers_$(arg ros2_control_command_interface).yaml"/>
+  <!-- Flag to preserve fixed joints and prevent lumping when generating SDF for Gazebo -->
+  <xacro:arg name="gazebo_preserve_fixed_joint" default="false"/>
+  <!--            -->
+  <!-- Properties -->
+  <!--            -->
+  <!-- Prefixes -->
+  <xacro:property name="prefix_arm" value="$(arg prefix)"/>
+  <xacro:property name="prefix_gripper" value="$(arg prefix)"/>
+  <!-- Origin of arm in the world -->
+  <xacro:property name="world_name" value="world"/>
+  <xacro:property name="origin_xyz" value="0 0 0"/>
+  <xacro:property name="origin_rpy" value="0 0 0"/>
+  <!-- Offset of gripper with respect to wrist flange -->
+  <xacro:property name="gripper_offset_xyz" value="0 0 0"/>
+  <xacro:property name="gripper_offset_rpy" value="0 0 0"/>
+  <!--       -->
+  <!-- Robot -->
+  <!--       -->
+  <!-- Dummy world link that the robot is fixed to -->
+  <xacro:panda_dummy_link
+    link_name="${world_name}"
+    gazebo_preserve_fixed_joint="$(arg gazebo_preserve_fixed_joint)"
+  />
+  <!-- Arm -->
+  <xacro:panda_arm
+    base_parent="world"
+    prefix="${prefix_arm}"
+    origin_xyz="${origin_xyz}"
+    origin_rpy="${origin_rpy}"
+    collision="$(arg collision_arm)"
+    safety_limits="$(arg safety_limits)"
+    safety_position_margin="$(arg safety_position_margin)"
+    safety_k_position="$(arg safety_k_position)"
+    safety_k_velocity="$(arg safety_k_velocity)"
+    ros2_control="$(arg ros2_control)"
+    ros2_control_plugin="$(arg ros2_control_plugin)"
+    ros2_control_command_interface="$(arg ros2_control_command_interface)"
+    gazebo_preserve_fixed_joint="$(arg gazebo_preserve_fixed_joint)"
+  />
+  <!-- Gripper -->
+  <xacro:if value="$(arg gripper)">
+    <xacro:panda_gripper
+      wrist_flange="${prefix_arm}${wrist_flange_name}"
+      prefix="${prefix_gripper}"
+      origin_xyz="${gripper_offset_xyz}"
+      origin_rpy="${gripper_offset_rpy}"
+      collision="$(arg collision_gripper)"
+      ros2_control="$(arg ros2_control)"
+      ros2_control_plugin="$(arg ros2_control_plugin)"
+      ros2_control_command_interface="$(arg ros2_control_command_interface)"
+      gazebo_preserve_fixed_joint="$(arg gazebo_preserve_fixed_joint)"
+    />
+  </xacro:if>
+  <!-- Gazebo - ROS 2 control (Ignition) -->
+  <xacro:if value="$(arg ros2_control)">
+    <xacro:if value="${'ign' in '$(arg ros2_control_plugin)'}">
+      <xacro:ign_ros2_control controller_parameters="$(arg ros2_controller_parameters)"/>
+    </xacro:if>
   </xacro:if>
 </robot>
